File: Cherry Mx Bitboard.kicad_pcb (KiCad board)
At the start: 2 copper layers, 19 x 19 mm, 12 parts, among them P11 CONN_01X01, P12 CONN_01X01, P13 CONN_01X01, P14 CONN_01X01, P15 CONN_01X01, P16 CONN_01X01, P21 CONN_01X01, P22 CONN_01X01, P23 CONN_01X01, P24 CONN_01X01, SW1 SW_PUSH

Commit message: initial
Routing:
- net /1: track 34.2 -> 15.0 mm
- net /2: track 31.3 -> 21.2 mm
Other:
- board size 19 x 19 mm -> 17.8 x 17.8 mm
Changed lines of the file:
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@@
-(kicad_pcb (version 4) (host pcbnew 4.0.2-stable)
+(kicad_pcb (version 4) (host pcbnew 4.0.7-e2-6376~61~ubuntu18.04.1)
   (general
     (links 11)
-    (no_connects 0)
-    (area 105.359999 99.009999 124.510001 118.160001)
+    (no_connects 6)
+    (area 102.862667 98.666 127.007334 118.604)
     (thickness 1.6)
-    (drawings 14)
-    (tracks 24)
+    (drawings 12)
+    (tracks 18)
     (zones 0)
     (modules 12)
@@
     (0 F.Cu signal)
     (31 B.Cu signal)
-    (32 B.Adhes user)
-    (33 F.Adhes user)
-    (34 B.Paste user)
-    (35 F.Paste user)
+    (32 B.Adhes user hide)
+    (33 F.Adhes user hide)
+    (34 B.Paste user hide)
+    (35 F.Paste user hide)
     (36 B.SilkS user)
     (37 F.SilkS user)
-    (38 B.Mask user)
-    (39 F.Mask user)
-    (40 Dwgs.User user)
-    (41 Cmts.User user)
-    (42 Eco1.User user)
-    (43 Eco2.User user)
+    (38 B.Mask user hide)
+    (39 F.Mask user hide)
+    (40 Dwgs.User user hide)
+    (41 Cmts.User user hide)
+    (42 Eco1.User user hide)
+    (43 Eco2.User user hide)
     (44 Edge.Cuts user)
-    (45 Margin user)
-    (46 B.CrtYd user)
-    (47 F.CrtYd user)
-    (48 B.Fab user)
-    (49 F.Fab user)
+    (45 Margin user hide)
+    (46 B.CrtYd user hide)
+    (47 F.CrtYd user hide)
+    (48 B.Fab user hide)
+    (49 F.Fab user hide)
   )
   (setup
@@
     (pad_to_mask_clearance 0)
     (aux_axis_origin 0 0)
-    (visible_elements 7FFEFF7F)
+    (visible_elements 7FFED479)
     (pcbplotparams
       (layerselection 0x00030_80000001)
@@
     (add_net "Net-(D1-Pad2)")
   )
+  (module footprint:switch (layer F.Cu)
+    (at 114.935 108.585)
+    (fp_text reference SW1 (at 0 3.429) (layer F.SilkS)
+      (effects (font (size 2 2) (thickness 0.2)))
+    )
+    (fp_text value SW_PUSH (at 0 -7.5) (layer F.Fab) hide
+      (effects (font (size 1 1) (thickness 0.15)))
+    )
+    (fp_line (start -6.5 -6.5) (end 6.5 -6.5) (layer F.SilkS) (width 0.15))
+    (fp_line (start 6.5 -6.5) (end 6.5 6.5) (layer F.SilkS) (width 0.15))
+    (fp_line (start 6.5 6.5) (end -6.5 6.5) (layer F.SilkS) (width 0.15))
+    (fp_line (start -6.5 6.5) (end -6.5 -6.5) (layer F.SilkS) (width 0.15))
+    (pad "" np_thru_hole circle (at 5.08 0) (size 1.71 1.71) (drill 1.71) (layers *.Cu *.Mask F.SilkS))
+    (pad 2 thru_hole circle (at 2.54 -5.08) (size 2.5 2.5) (drill 1.5) (layers *.Cu *.Mask F.SilkS)
+      (net 1 "Net-(D1-Pad2)"))
+    (pad "" np_thru_hole circle (at 0 0) (size 4 4) (drill 4) (layers *.Cu *.Mask F.SilkS))
+    (pad 1 thru_hole circle (at -3.81 -2.54) (size 2.5 2.5) (drill 1.5) (layers *.Cu *.Mask F.SilkS)
+      (net 3 /1))
+    (pad "" np_thru_hole circle (at -5.08 0) (size 1.71 1.71) (drill 1.71) (layers *.Cu *.Mask F.SilkS))
+  )
   (module footprint:diode (layer B.Cu)
     (at 115.57 100.965)
@@
       (net 2 /2))
   )
-  (module footprint:switch (layer F.Cu)
-    (at 114.935 108.585)
-    (fp_text reference SW1 (at 0 3.429) (layer F.SilkS)
-      (effects (font (size 2 2) (thickness 0.2)))
-    )
-    (fp_text value SW_PUSH (at 0 -7.5) (layer F.Fab) hide
-      (effects (font (size 1 1) (thickness 0.15)))
-    )
-    (fp_line (start -6.5 -6.5) (end 6.5 -6.5) (layer F.SilkS) (width 0.15))
-    (fp_line (start 6.5 -6.5) (end 6.5 6.5) (layer F.SilkS) (width 0.15))
-    (fp_line (start 6.5 6.5) (end -6.5 6.5) (layer F.SilkS) (width 0.15))
-    (fp_line (start -6.5 6.5) (end -6.5 -6.5) (layer F.SilkS) (width 0.15))
-    (pad "" np_thru_hole circle (at 5.08 0) (size 1.71 1.71) (drill 1.71) (layers *.Cu *.Mask F.SilkS))
-    (pad 2 thru_hole circle (at 2.54 -5.08) (size 2.5 2.5) (drill 1.5) (layers *.Cu *.Mask F.SilkS)
-      (net 1 "Net-(D1-Pad2)"))
-    (pad "" np_thru_hole circle (at 0 0) (size 4 4) (drill 4) (layers *.Cu *.Mask F.SilkS))
-    (pad 1 thru_hole circle (at -3.81 -2.54) (size 2.5 2.5) (drill 1.5) (layers *.Cu *.Mask F.SilkS)
-      (net 3 /1))
-    (pad "" np_thru_hole circle (at -5.08 0) (size 1.71 1.71) (drill 1.71) (layers *.Cu *.Mask F.SilkS))
-    (pad "" np_thru_hole circle (at 1.27 5.08) (size 0.8 0.8) (drill 0.8) (layers *.Cu *.Mask F.SilkS))
-    (pad "" np_thru_hole circle (at -1.27 5.08) (size 0.8 0.8) (drill 0.8) (layers *.Cu *.Mask F.SilkS))
-  )
-  (gr_text 2 (at 106.172 111.125) (layer B.SilkS)
+  (gr_line (start 113.3 114.7) (end 116.75 114.7) (angle 90) (layer Edge.Cuts) (width 0.1))
+  (gr_line (start 116.75 114.7) (end 116.75 111.2) (angle 90) (layer Edge.Cuts) (width 0.1))
+  (gr_line (start 113.3 114.7) (end 113.3 111.2) (angle 90) (layer Edge.Cuts) (width 0.1))
+  (gr_line (start 113.3 111.2) (end 116.75 111.2) (angle 90) (layer Edge.Cuts) (width 0.1))
+  (gr_line (start 123.825 99.695) (end 106.045 99.695) (angle 90) (layer Edge.Cuts) (width 0.1))
+  (gr_line (start 123.825 117.475) (end 123.825 99.695) (angle 90) (layer Edge.Cuts) (width 0.1))
+  (gr_line (start 106.045 117.475) (end 123.825 117.475) (angle 90) (layer Edge.Cuts) (width 0.1))
+  (gr_line (start 106.045 99.695) (end 106.045 117.475) (angle 90) (layer Edge.Cuts) (width 0.1))
+  (gr_text 1 (at 111.125 116.84) (layer B.SilkS)
     (effects (font (size 1.2 1.2) (thickness 0.2)) (justify mirror))
   )
-  (gr_text 2 (at 106.172 106.045) (layer B.SilkS)
+  (gr_text 2 (at 106.68 104.14) (layer B.SilkS)
     (effects (font (size 1.2 1.2) (thickness 0.2)) (justify mirror))
   )
-  (gr_text 1 (at 109.22 116.84) (layer B.SilkS)
-    (effects (font (size 1.2 1.2) (thickness 0.2)) (justify mirror))
-  )
-  (gr_text 1 (at 106.299 100.457) (layer B.SilkS)
-    (effects (font (size 1.2 1.2) (thickness 0.2)) (justify mirror))
-  )
-  (gr_text 1 (at 113.665 116.84) (layer B.SilkS)
-    (effects (font (size 1.2 1.2) (thickness 0.2)) (justify mirror))
-  )
-  (gr_text 1 (at 118.745 116.84) (layer B.SilkS)
-    (effects (font (size 1.2 1.2) (thickness 0.2)) (justify mirror))
-  )
-  (gr_text 1 (at 123.19 116.84) (layer B.SilkS)
-    (effects (font (size 1.2 1.2) (thickness 0.2)) (justify mirror))
-  )
-  (gr_text 2 (at 123.698 111.125) (layer B.SilkS)
-    (effects (font (size 1.2 1.2) (thickness 0.2)) (justify mirror))
-  )
-  (gr_text 2 (at 123.698 106.045) (layer B.SilkS)
+  (gr_text 2 (at 123.19 104.14) (layer B.SilkS)
     (effects (font (size 1.2 1.2) (thickness 0.2)) (justify mirror))
   )
@@
     (effects (font (size 1.2 1.2) (thickness 0.2)) (justify mirror))
   )
-  (gr_line (start 105.41 118.11) (end 105.41 99.06) (angle 90) (layer Edge.Cuts) (width 0.1))
-  (gr_line (start 124.46 118.11) (end 105.41 118.11) (angle 90) (layer Edge.Cuts) (width 0.1))
-  (gr_line (start 124.46 99.06) (end 124.46 118.11) (angle 90) (layer Edge.Cuts) (width 0.1))
-  (gr_line (start 105.41 99.06) (end 124.46 99.06) (angle 90) (layer Edge.Cuts) (width 0.1))
   (segment (start 117.475 103.505) (end 120.015 103.505) (width 0.4) (layer F.Cu) (net 1))
   (segment (start 120.015 103.505) (end 121.92 101.6) (width 0.4) (layer F.Cu) (net 1))
   (segment (start 121.92 101.6) (end 121.92 100.965) (width 0.4) (layer F.Cu) (net 1))
-  (segment (start 121.92 106.045) (end 121.92 111.125) (width 0.4) (layer B.Cu) (net 2))
-  (segment (start 107.95 106.045) (end 107.95 111.125) (width 0.4) (layer B.Cu) (net 2))
   (segment (start 115.57 100.965) (end 115.57 101.6) (width 0.4) (layer B.Cu) (net 2))
   (segment (start 115.57 101.6) (end 113.665 103.505) (width 0.4) (layer B.Cu) (net 2))
@@
   (segment (start 121.92 103.505) (end 121.92 106.045) (width 0.4) (layer B.Cu) (net 2))
   (segment (start 119.38 100.965) (end 121.92 103.505) (width 0.4) (layer B.Cu) (net 2))
+  (segment (start 112.395 101.6) (end 112.395 104.775) (width 0.4) (layer F.Cu) (net 3))
+  (segment (start 112.395 104.775) (end 111.125 106.045) (width 0.4) (layer F.Cu) (net 3))
   (segment (start 111.125 106.045) (end 111.125 106.68) (width 0.4) (layer F.Cu) (net 3))
   (segment (start 111.125 106.68) (end 111.76 107.315) (width 0.4) (layer F.Cu) (net 3))
@@
   (segment (start 111.76 113.03) (end 112.395 113.665) (width 0.4) (layer F.Cu) (net 3))
   (segment (start 111.76 107.315) (end 111.76 113.03) (width 0.4) (layer F.Cu) (net 3))
-  (segment (start 117.475 115.57) (end 121.92 115.57) (width 0.4) (layer F.Cu) (net 3))
-  (segment (start 112.395 115.57) (end 117.475 115.57) (width 0.4) (layer F.Cu) (net 3))
-  (segment (start 107.95 115.57) (end 112.395 115.57) (width 0.4) (layer F.Cu) (net 3))
-  (segment (start 112.395 101.6) (end 107.95 101.6) (width 0.4) (layer F.Cu) (net 3))
-  (segment (start 107.95 101.6) (end 107.95 102.87) (width 0.4) (layer F.Cu) (net 3))
-  (segment (start 107.95 102.87) (end 111.125 106.045) (width 0.4) (layer F.Cu) (net 3))
 )

Commit message: first orderd
Parts:
- added A: CONN_01X01, MYLIB:1PIN_0.1, F.Cu at (170.8, 88.3)
- added A: CONN_01X01, MYLIB:1PIN_0.1, F.Cu at (160.7, 92.7)
- added D1: D, footprint:diode, B.Cu at (165.1, 120.0)
- added D1: D, footprint:diode, B.Cu at (91.4, 101.6)
- added D1: D, footprint:diode, B.Cu at (146.7, 83.2)
- added D1: D, footprint:diode, B.Cu at (128.3, 83.2)
- added D1: D, footprint:diode, B.Cu at (109.9, 83.2)
- added D1: D, footprint:diode, B.Cu at (91.4, 83.2)
- added D1: D, footprint:diode, B.Cu at (146.7, 64.8)
- added D1: D, footprint:diode, B.Cu at (128.3, 64.8)
- added D1: D, footprint:diode, B.Cu at (109.9, 64.8)
- added D1: D, footprint:diode, B.Cu at (91.4, 64.8)
- added D1: D, footprint:diode, B.Cu at (146.7, 46.4)
- added D1: D, footprint:diode, B.Cu at (165.1, 101.6)
- added D1: D, footprint:diode, B.Cu at (128.3, 46.4)
- added D1: D, footprint:diode, B.Cu at (109.9, 46.4)
- added D1: D, footprint:diode, B.Cu at (146.7, 120.0)
- added D1: D, footprint:diode, B.Cu at (128.3, 120.0)
- added D1: D, footprint:diode, B.Cu at (109.9, 120.0)
- added D1: D, footprint:diode, B.Cu at (91.4, 120.0)
- added D1: D, footprint:diode, B.Cu at (146.7, 101.6)
- added D1: D, footprint:diode, B.Cu at (128.3, 101.6)
- added D1: D, footprint:diode, B.Cu at (109.9, 101.6)
- added DATA: CONN_01X01, MYLIB:1PIN_0.1, F.Cu at (173.4, 88.3)
- added DATA: CONN_01X01, MYLIB:1PIN_0.1, F.Cu at (157.5, 92.7)
- added DT: CONN_01X01, MYLIB:1PIN_0.1, F.Cu at (167.6, 51.4)
- added HOLE_M2: VAL**, MYLIB:HOLE_M2, F.Cu at (172.7, 80.0)
- added HOLE_M2: VAL**, MYLIB:HOLE_M2, F.Cu at (158.8, 80.0)
- added HOLE_M2: VAL**, MYLIB:HOLE_M2, F.Cu at (173.4, 96.5)
- added HOLE_M2: VAL**, MYLIB:HOLE_M2, F.Cu at (157.5, 96.5)
- added JACK: MJ-4PP-9, MYLIB_REV:MJ-4PP-9_rev2, F.Cu at (155.6, 89.5)
- added JACK: MJ-4PP-9, MYLIB_REV:MJ-4PP-9_rev2, F.Cu at (175.8, 91.2)
- added OLED: OLED, MYLIB:MY_SIL-4, F.Cu at (161.9, 80.0)
- added P11: CONN_01X01, footprint:wirepad, F.Cu at (161.9, 120.0)
- added P11: CONN_01X01, footprint:wirepad, F.Cu at (88.3, 101.6)
- added P11: CONN_01X01, footprint:wirepad, F.Cu at (143.5, 83.2)
- added P11: CONN_01X01, footprint:wirepad, F.Cu at (125.1, 83.2)
- added P11: CONN_01X01, footprint:wirepad, F.Cu at (106.7, 83.2)
- added P11: CONN_01X01, footprint:wirepad, F.Cu at (88.3, 83.2)
- added P11: CONN_01X01, footprint:wirepad, F.Cu at (143.5, 64.8)
- added P11: CONN_01X01, footprint:wirepad, F.Cu at (125.1, 64.8)
- added P11: CONN_01X01, footprint:wirepad, F.Cu at (106.7, 64.8)
- added P11: CONN_01X01, footprint:wirepad, F.Cu at (88.3, 64.8)
- added P11: CONN_01X01, footprint:wirepad, F.Cu at (143.5, 46.4)
- added P11: CONN_01X01, footprint:wirepad, F.Cu at (161.9, 101.6)
- added P11: CONN_01X01, footprint:wirepad, F.Cu at (125.1, 46.4)
- added P11: CONN_01X01, footprint:wirepad, F.Cu at (106.7, 46.4)
- added P11: CONN_01X01, footprint:wirepad, F.Cu at (143.5, 120.0)
- added P11: CONN_01X01, footprint:wirepad, F.Cu at (125.1, 120.0)
- added P11: CONN_01X01, footprint:wirepad, F.Cu at (106.7, 120.0)
- added P11: CONN_01X01, footprint:wirepad, F.Cu at (88.3, 120.0)
- added P11: CONN_01X01, footprint:wirepad, F.Cu at (143.5, 101.6)
- added P11: CONN_01X01, footprint:wirepad, F.Cu at (125.1, 101.6)
- added P11: CONN_01X01, footprint:wirepad, F.Cu at (106.7, 101.6)
- added P12: CONN_01X01, footprint:wirepad, F.Cu at (156.8, 125.1)
- added P12: CONN_01X01, footprint:wirepad, F.Cu at (83.2, 106.7)
- added P12: CONN_01X01, footprint:wirepad, F.Cu at (138.4, 88.3)
- added P12: CONN_01X01, footprint:wirepad, F.Cu at (120.0, 88.3)
- added P12: CONN_01X01, footprint:wirepad, F.Cu at (101.6, 88.3)
- added P12: CONN_01X01, footprint:wirepad, F.Cu at (83.2, 88.3)
- added P12: CONN_01X01, footprint:wirepad, F.Cu at (138.4, 69.8)
- added P12: CONN_01X01, footprint:wirepad, F.Cu at (120.0, 69.8)
- added P12: CONN_01X01, footprint:wirepad, F.Cu at (101.6, 69.8)
- added P12: CONN_01X01, footprint:wirepad, F.Cu at (83.2, 69.8)
- added P12: CONN_01X01, footprint:wirepad, F.Cu at (138.4, 51.4)
- added P12: CONN_01X01, footprint:wirepad, F.Cu at (156.8, 106.7)
- added P12: CONN_01X01, footprint:wirepad, F.Cu at (120.0, 51.4)
- added P12: CONN_01X01, footprint:wirepad, F.Cu at (101.6, 51.4)
- added P12: CONN_01X01, footprint:wirepad, F.Cu at (138.4, 125.1)
- added P12: CONN_01X01, footprint:wirepad, F.Cu at (120.0, 125.1)
- added P12: CONN_01X01, footprint:wirepad, F.Cu at (101.6, 125.1)
- added P12: CONN_01X01, footprint:wirepad, F.Cu at (83.2, 125.1)
- added P12: CONN_01X01, footprint:wirepad, F.Cu at (138.4, 106.7)
- added P12: CONN_01X01, footprint:wirepad, F.Cu at (120.0, 106.7)
- added P12: CONN_01X01, footprint:wirepad, F.Cu at (101.6, 106.7)
- added P13: CONN_01X01, footprint:wirepad, F.Cu at (161.9, 116.8)
- added P13: CONN_01X01, footprint:wirepad, F.Cu at (88.3, 116.8)
- added P13: CONN_01X01, footprint:wirepad, F.Cu at (143.5, 98.4)
- added P13: CONN_01X01, footprint:wirepad, F.Cu at (125.1, 98.4)
- added P13: CONN_01X01, footprint:wirepad, F.Cu at (106.7, 98.4)
- added P13: CONN_01X01, footprint:wirepad, F.Cu at (88.3, 98.4)
- added P13: CONN_01X01, footprint:wirepad, F.Cu at (143.5, 80.0)
- added P13: CONN_01X01, footprint:wirepad, F.Cu at (125.1, 80.0)
- added P13: CONN_01X01, footprint:wirepad, F.Cu at (106.7, 80.0)
- added P13: CONN_01X01, footprint:wirepad, F.Cu at (88.3, 80.0)
- added P13: CONN_01X01, footprint:wirepad, F.Cu at (143.5, 61.6)
- added P13: CONN_01X01, footprint:wirepad, F.Cu at (161.9, 135.3)
- added P13: CONN_01X01, footprint:wirepad, F.Cu at (125.1, 61.6)
- added P13: CONN_01X01, footprint:wirepad, F.Cu at (106.7, 61.6)
- added P13: CONN_01X01, footprint:wirepad, F.Cu at (143.5, 135.3)
- added P13: CONN_01X01, footprint:wirepad, F.Cu at (125.1, 135.3)
- added P13: CONN_01X01, footprint:wirepad, F.Cu at (106.7, 135.3)
- added P13: CONN_01X01, footprint:wirepad, F.Cu at (88.3, 135.3)
- added P13: CONN_01X01, footprint:wirepad, F.Cu at (143.5, 116.8)
- added P13: CONN_01X01, footprint:wirepad, F.Cu at (125.1, 116.8)
- added P13: CONN_01X01, footprint:wirepad, F.Cu at (106.7, 116.8)
- added P14: CONN_01X01, footprint:wirepad, F.Cu at (156.8, 116.8)
- added P14: CONN_01X01, footprint:wirepad, F.Cu at (83.2, 116.8)
- added P14: CONN_01X01, footprint:wirepad, F.Cu at (138.4, 98.4)
- added P14: CONN_01X01, footprint:wirepad, F.Cu at (120.0, 98.4)
- added P14: CONN_01X01, footprint:wirepad, F.Cu at (101.6, 98.4)
- added P14: CONN_01X01, footprint:wirepad, F.Cu at (83.2, 98.4)
- added P14: CONN_01X01, footprint:wirepad, F.Cu at (138.4, 80.0)
- added P14: CONN_01X01, footprint:wirepad, F.Cu at (120.0, 80.0)
- added P14: CONN_01X01, footprint:wirepad, F.Cu at (101.6, 80.0)
- added P14: CONN_01X01, footprint:wirepad, F.Cu at (83.2, 80.0)
- added P14: CONN_01X01, footprint:wirepad, F.Cu at (138.4, 61.6)
- added P14: CONN_01X01, footprint:wirepad, F.Cu at (156.8, 135.3)
- added P14: CONN_01X01, footprint:wirepad, F.Cu at (120.0, 61.6)
- added P14: CONN_01X01, footprint:wirepad, F.Cu at (101.6, 61.6)
- added P14: CONN_01X01, footprint:wirepad, F.Cu at (138.4, 135.3)
- added P14: CONN_01X01, footprint:wirepad, F.Cu at (120.0, 135.3)
- added P14: CONN_01X01, footprint:wirepad, F.Cu at (101.6, 135.3)
- added P14: CONN_01X01, footprint:wirepad, F.Cu at (83.2, 135.3)
- added P14: CONN_01X01, footprint:wirepad, F.Cu at (138.4, 116.8)
- added P14: CONN_01X01, footprint:wirepad, F.Cu at (120.0, 116.8)
- added P14: CONN_01X01, footprint:wirepad, F.Cu at (101.6, 116.8)
- added P15: CONN_01X01, footprint:wirepad, F.Cu at (172.1, 116.8)
- added P15: CONN_01X01, footprint:wirepad, F.Cu at (98.4, 116.8)
- added P15: CONN_01X01, footprint:wirepad, F.Cu at (153.7, 98.4)
- added P15: CONN_01X01, footprint:wirepad, F.Cu at (135.3, 98.4)
- added P15: CONN_01X01, footprint:wirepad, F.Cu at (116.8, 98.4)
- added P15: CONN_01X01, footprint:wirepad, F.Cu at (98.4, 98.4)
- added P15: CONN_01X01, footprint:wirepad, F.Cu at (153.7, 80.0)
- added P15: CONN_01X01, footprint:wirepad, F.Cu at (135.3, 80.0)
- added P15: CONN_01X01, footprint:wirepad, F.Cu at (116.8, 80.0)
- added P15: CONN_01X01, footprint:wirepad, F.Cu at (98.4, 80.0)
- added P15: CONN_01X01, footprint:wirepad, F.Cu at (153.7, 61.6)
- added P15: CONN_01X01, footprint:wirepad, F.Cu at (172.1, 135.3)
- added P15: CONN_01X01, footprint:wirepad, F.Cu at (135.3, 61.6)
- added P15: CONN_01X01, footprint:wirepad, F.Cu at (116.8, 61.6)
- added P15: CONN_01X01, footprint:wirepad, F.Cu at (153.7, 135.3)
- added P15: CONN_01X01, footprint:wirepad, F.Cu at (135.3, 135.3)
- added P15: CONN_01X01, footprint:wirepad, F.Cu at (116.8, 135.3)
- added P15: CONN_01X01, footprint:wirepad, F.Cu at (98.4, 135.3)
- added P15: CONN_01X01, footprint:wirepad, F.Cu at (153.7, 116.8)
- added P15: CONN_01X01, footprint:wirepad, F.Cu at (135.3, 116.8)
- added P15: CONN_01X01, footprint:wirepad, F.Cu at (116.8, 116.8)
- added P16: CONN_01X01, footprint:wirepad, F.Cu at (167.0, 116.8)
- added P16: CONN_01X01, footprint:wirepad, F.Cu at (93.3, 116.8)
- added P16: CONN_01X01, footprint:wirepad, F.Cu at (148.6, 98.4)
- added P16: CONN_01X01, footprint:wirepad, F.Cu at (130.2, 98.4)
- added P16: CONN_01X01, footprint:wirepad, F.Cu at (111.8, 98.4)
- added P16: CONN_01X01, footprint:wirepad, F.Cu at (93.3, 98.4)
- added P16: CONN_01X01, footprint:wirepad, F.Cu at (148.6, 80.0)
- added P16: CONN_01X01, footprint:wirepad, F.Cu at (130.2, 80.0)
- added P16: CONN_01X01, footprint:wirepad, F.Cu at (111.8, 80.0)
- added P16: CONN_01X01, footprint:wirepad, F.Cu at (93.3, 80.0)
- added P16: CONN_01X01, footprint:wirepad, F.Cu at (148.6, 61.6)
- added P16: CONN_01X01, footprint:wirepad, F.Cu at (167.0, 135.3)
- added P16: CONN_01X01, footprint:wirepad, F.Cu at (130.2, 61.6)
- added P16: CONN_01X01, footprint:wirepad, F.Cu at (111.8, 61.6)
- added P16: CONN_01X01, footprint:wirepad, F.Cu at (148.6, 135.3)
- added P16: CONN_01X01, footprint:wirepad, F.Cu at (130.2, 135.3)
- added P16: CONN_01X01, footprint:wirepad, F.Cu at (111.8, 135.3)
- added P16: CONN_01X01, footprint:wirepad, F.Cu at (93.3, 135.3)
- added P16: CONN_01X01, footprint:wirepad, F.Cu at (148.6, 116.8)
- added P16: CONN_01X01, footprint:wirepad, F.Cu at (130.2, 116.8)
- added P16: CONN_01X01, footprint:wirepad, F.Cu at (111.8, 116.8)
- added P2: CONN_01X01, MYLIB:1PIN_0.1, F.Cu at (173.4, 85.1)
- added P2: CONN_01X01, MYLIB:1PIN_0.1, F.Cu at (167.6, 64.1)
- added P2: CONN_01X01, MYLIB:1PIN_0.1, F.Cu at (167.6, 66.7)
- added P2: CONN_01X01, MYLIB:1PIN_0.1, F.Cu at (170.2, 69.2)
- added P2: CONN_01X01, MYLIB:1PIN_0.1, F.Cu at (167.6, 69.2)
- added P2: CONN_01X01, MYLIB:1PIN_0.1, F.Cu at (170.2, 64.1)
- added P2: CONN_01X01, MYLIB:1PIN_0.1, F.Cu at (170.2, 71.8)
- added P2: CONN_01X01, MYLIB:1PIN_0.1, F.Cu at (167.6, 71.8)
- added P2: CONN_01X01, MYLIB:1PIN_0.1, F.Cu at (170.2, 74.3)
- added P2: CONN_01X01, MYLIB:1PIN_0.1, F.Cu at (167.6, 74.3)
- added P2: CONN_01X01, MYLIB:1PIN_0.1, F.Cu at (170.2, 76.8)
- added P2: CONN_01X01, MYLIB:1PIN_0.1, F.Cu at (170.8, 85.1)
- added P2: CONN_01X01, MYLIB:1PIN_0.1, F.Cu at (167.6, 76.8)
- added P2: CONN_01X01, MYLIB:1PIN_0.1, F.Cu at (161.3, 74.3)
- added P2: CONN_01X01, MYLIB:1PIN_0.1, F.Cu at (163.8, 76.8)
- added P2: CONN_01X01, MYLIB:1PIN_0.1, F.Cu at (163.8, 74.3)
- added P2: CONN_01X01, MYLIB:1PIN_0.1, F.Cu at (163.8, 71.8)
- added P2: CONN_01X01, MYLIB:1PIN_0.1, F.Cu at (161.3, 71.8)
- added P2: CONN_01X01, MYLIB:1PIN_0.1, F.Cu at (161.3, 76.8)
- added P2: CONN_01X01, MYLIB:1PIN_0.1, F.Cu at (161.3, 69.2)
- added P2: CONN_01X01, MYLIB:1PIN_0.1, F.Cu at (163.8, 69.2)
- added P2: CONN_01X01, MYLIB:1PIN_0.1, F.Cu at (161.3, 66.7)
- added P2: CONN_01X01, MYLIB:1PIN_0.1, F.Cu at (170.8, 82.5)
- added P2: CONN_01X01, MYLIB:1PIN_0.1, F.Cu at (163.8, 66.7)
- added P2: CONN_01X01, MYLIB:1PIN_0.1, F.Cu at (161.3, 64.1)
- added P2: CONN_01X01, MYLIB:1PIN_0.1, F.Cu at (163.8, 64.1)
- added P2: CONN_01X01, MYLIB:1PIN_0.1, F.Cu at (161.3, 61.6)
- added P2: CONN_01X01, MYLIB:1PIN_0.1, F.Cu at (167.6, 59.1)
- added P2: CONN_01X01, MYLIB:1PIN_0.1, F.Cu at (167.6, 61.6)
- added P2: CONN_01X01, MYLIB:1PIN_0.1, F.Cu at (167.6, 48.9)
- added P2: CONN_01X01, MYLIB:1PIN_0.1, F.Cu at (167.6, 54.0)
- added P2: CONN_01X01, MYLIB:1PIN_0.1, F.Cu at (167.6, 56.5)
- added P2: CONN_01X01, MYLIB:1PIN_0.1, F.Cu at (163.8, 59.1)
- added P2: CONN_01X01, MYLIB:1PIN_0.1, F.Cu at (173.4, 82.5)
- added P2: CONN_01X01, MYLIB:1PIN_0.1, F.Cu at (163.8, 61.6)
- added P2: CONN_01X01, MYLIB:1PIN_0.1, F.Cu at (163.8, 48.9)
- added P2: CONN_01X01, MYLIB:1PIN_0.1, F.Cu at (163.8, 54.0)
- added P2: CONN_01X01, MYLIB:1PIN_0.1, F.Cu at (163.8, 56.5)
- added P2: CONN_01X01, MYLIB:1PIN_0.1, F.Cu at (163.8, 51.4)
- added P2: CONN_01X01, MYLIB:1PIN_0.1, F.Cu at (170.2, 61.6)
- added P2: CONN_01X01, MYLIB:1PIN_0.1, F.Cu at (170.2, 48.9)
- added P2: CONN_01X01, MYLIB:1PIN_0.1, F.Cu at (170.2, 59.1)
- added P2: CONN_01X01, MYLIB:1PIN_0.1, F.Cu at (170.2, 54.0)
- added P2: CONN_01X01, MYLIB:1PIN_0.1, F.Cu at (170.2, 51.4)
- added P2: CONN_01X01, MYLIB:1PIN_0.1, F.Cu at (158.1, 85.1)
- added P2: CONN_01X01, MYLIB:1PIN_0.1, F.Cu at (170.2, 56.5)
- added P2: CONN_01X01, MYLIB:1PIN_0.1, F.Cu at (161.3, 59.1)
- added P2: CONN_01X01, MYLIB:1PIN_0.1, F.Cu at (161.3, 56.5)
- added P2: CONN_01X01, MYLIB:1PIN_0.1, F.Cu at (161.3, 54.0)
- added P2: CONN_01X01, MYLIB:1PIN_0.1, F.Cu at (161.3, 51.4)
- added P2: CONN_01X01, MYLIB:1PIN_0.1, F.Cu at (161.3, 48.9)
- added P2: CONN_01X01, MYLIB:1PIN_0.1, F.Cu at (160.7, 85.1)
- added P2: CONN_01X01, MYLIB:1PIN_0.1, F.Cu at (158.1, 82.5)
- added P2: CONN_01X01, MYLIB:1PIN_0.1, F.Cu at (160.7, 82.5)
- added P2: CONN_01X01, MYLIB:1PIN_0.1, F.Cu at (170.2, 66.7)
- added P21: CONN_01X01, footprint:wirepad, F.Cu at (172.1, 111.8)
- added P21: CONN_01X01, footprint:wirepad, F.Cu at (98.4, 111.8)
- added P21: CONN_01X01, footprint:wirepad, F.Cu at (153.7, 93.3)
- added P21: CONN_01X01, footprint:wirepad, F.Cu at (135.3, 93.3)
- added P21: CONN_01X01, footprint:wirepad, F.Cu at (116.8, 93.3)
- added P21: CONN_01X01, footprint:wirepad, F.Cu at (98.4, 93.3)
- added P21: CONN_01X01, footprint:wirepad, F.Cu at (153.7, 74.9)
- added P21: CONN_01X01, footprint:wirepad, F.Cu at (135.3, 74.9)
- added P21: CONN_01X01, footprint:wirepad, F.Cu at (116.8, 74.9)
- added P21: CONN_01X01, footprint:wirepad, F.Cu at (98.4, 74.9)
- added P21: CONN_01X01, footprint:wirepad, F.Cu at (153.7, 56.5)
- added P21: CONN_01X01, footprint:wirepad, F.Cu at (172.1, 130.2)
- added P21: CONN_01X01, footprint:wirepad, F.Cu at (135.3, 56.5)
- added P21: CONN_01X01, footprint:wirepad, F.Cu at (116.8, 56.5)
- added P21: CONN_01X01, footprint:wirepad, F.Cu at (153.7, 130.2)
- added P21: CONN_01X01, footprint:wirepad, F.Cu at (135.3, 130.2)
- added P21: CONN_01X01, footprint:wirepad, F.Cu at (116.8, 130.2)
- added P21: CONN_01X01, footprint:wirepad, F.Cu at (98.4, 130.2)
- added P21: CONN_01X01, footprint:wirepad, F.Cu at (153.7, 111.8)
- added P21: CONN_01X01, footprint:wirepad, F.Cu at (135.3, 111.8)
- added P21: CONN_01X01, footprint:wirepad, F.Cu at (116.8, 111.8)
- added P22: CONN_01X01, footprint:wirepad, F.Cu at (172.1, 106.7)
- added P22: CONN_01X01, footprint:wirepad, F.Cu at (98.4, 106.7)
- added P22: CONN_01X01, footprint:wirepad, F.Cu at (153.7, 88.3)
- added P22: CONN_01X01, footprint:wirepad, F.Cu at (135.3, 88.3)
- added P22: CONN_01X01, footprint:wirepad, F.Cu at (116.8, 88.3)
- added P22: CONN_01X01, footprint:wirepad, F.Cu at (98.4, 88.3)
- added P22: CONN_01X01, footprint:wirepad, F.Cu at (153.7, 69.8)
- added P22: CONN_01X01, footprint:wirepad, F.Cu at (135.3, 69.8)
- added P22: CONN_01X01, footprint:wirepad, F.Cu at (116.8, 69.8)
- added P22: CONN_01X01, footprint:wirepad, F.Cu at (98.4, 69.8)
- added P22: CONN_01X01, footprint:wirepad, F.Cu at (153.7, 51.4)
- added P22: CONN_01X01, footprint:wirepad, F.Cu at (172.1, 125.1)
- added P22: CONN_01X01, footprint:wirepad, F.Cu at (135.3, 51.4)
- added P22: CONN_01X01, footprint:wirepad, F.Cu at (116.8, 51.4)
- added P22: CONN_01X01, footprint:wirepad, F.Cu at (153.7, 125.1)
- added P22: CONN_01X01, footprint:wirepad, F.Cu at (135.3, 125.1)
- added P22: CONN_01X01, footprint:wirepad, F.Cu at (116.8, 125.1)
- added P22: CONN_01X01, footprint:wirepad, F.Cu at (98.4, 125.1)
- added P22: CONN_01X01, footprint:wirepad, F.Cu at (153.7, 106.7)
- added P22: CONN_01X01, footprint:wirepad, F.Cu at (135.3, 106.7)
- added P22: CONN_01X01, footprint:wirepad, F.Cu at (116.8, 106.7)
- added P23: CONN_01X01, footprint:wirepad, F.Cu at (156.8, 120.0)
- added P23: CONN_01X01, footprint:wirepad, F.Cu at (83.2, 101.6)
- added P23: CONN_01X01, footprint:wirepad, F.Cu at (138.4, 83.2)
- added P23: CONN_01X01, footprint:wirepad, F.Cu at (120.0, 83.2)
- added P23: CONN_01X01, footprint:wirepad, F.Cu at (101.6, 83.2)
- added P23: CONN_01X01, footprint:wirepad, F.Cu at (83.2, 83.2)
- added P23: CONN_01X01, footprint:wirepad, F.Cu at (138.4, 64.8)
- added P23: CONN_01X01, footprint:wirepad, F.Cu at (120.0, 64.8)
- added P23: CONN_01X01, footprint:wirepad, F.Cu at (101.6, 64.8)
- added P23: CONN_01X01, footprint:wirepad, F.Cu at (83.2, 64.8)
- added P23: CONN_01X01, footprint:wirepad, F.Cu at (138.4, 46.4)
- added P23: CONN_01X01, footprint:wirepad, F.Cu at (156.8, 101.6)
- added P23: CONN_01X01, footprint:wirepad, F.Cu at (120.0, 46.4)
- added P23: CONN_01X01, footprint:wirepad, F.Cu at (101.6, 46.4)
- added P23: CONN_01X01, footprint:wirepad, F.Cu at (138.4, 120.0)
- added P23: CONN_01X01, footprint:wirepad, F.Cu at (120.0, 120.0)
- added P23: CONN_01X01, footprint:wirepad, F.Cu at (101.6, 120.0)
- added P23: CONN_01X01, footprint:wirepad, F.Cu at (83.2, 120.0)
- added P23: CONN_01X01, footprint:wirepad, F.Cu at (138.4, 101.6)
- added P23: CONN_01X01, footprint:wirepad, F.Cu at (120.0, 101.6)
- added P23: CONN_01X01, footprint:wirepad, F.Cu at (101.6, 101.6)
- added P24: CONN_01X01, footprint:wirepad, F.Cu at (156.8, 130.2)
- added P24: CONN_01X01, footprint:wirepad, F.Cu at (83.2, 111.8)
- added P24: CONN_01X01, footprint:wirepad, F.Cu at (138.4, 93.3)
- added P24: CONN_01X01, footprint:wirepad, F.Cu at (120.0, 93.3)
- added P24: CONN_01X01, footprint:wirepad, F.Cu at (101.6, 93.3)
- added P24: CONN_01X01, footprint:wirepad, F.Cu at (83.2, 93.3)
- added P24: CONN_01X01, footprint:wirepad, F.Cu at (138.4, 74.9)
- added P24: CONN_01X01, footprint:wirepad, F.Cu at (120.0, 74.9)
- added P24: CONN_01X01, footprint:wirepad, F.Cu at (101.6, 74.9)
- added P24: CONN_01X01, footprint:wirepad, F.Cu at (83.2, 74.9)
- added P24: CONN_01X01, footprint:wirepad, F.Cu at (138.4, 56.5)
- added P24: CONN_01X01, footprint:wirepad, F.Cu at (156.8, 111.8)
- added P24: CONN_01X01, footprint:wirepad, F.Cu at (120.0, 56.5)
- added P24: CONN_01X01, footprint:wirepad, F.Cu at (101.6, 56.5)
- added P24: CONN_01X01, footprint:wirepad, F.Cu at (138.4, 130.2)
- added P24: CONN_01X01, footprint:wirepad, F.Cu at (120.0, 130.2)
- added P24: CONN_01X01, footprint:wirepad, F.Cu at (101.6, 130.2)
- added P24: CONN_01X01, footprint:wirepad, F.Cu at (83.2, 130.2)
- added P24: CONN_01X01, footprint:wirepad, F.Cu at (138.4, 111.8)
- added P24: CONN_01X01, footprint:wirepad, F.Cu at (120.0, 111.8)
- added P24: CONN_01X01, footprint:wirepad, F.Cu at (101.6, 111.8)
- added RESET1: RESET, MYLIB:SW_3.5x6.0_TH, F.Cu at (165.8, 83.8)
- added SW1: SW_PUSH, footprint:switch, F.Cu at (164.5, 109.2)
- added SW1: SW_PUSH, footprint:switch, F.Cu at (90.8, 109.2)
- added SW1: SW_PUSH, footprint:switch, F.Cu at (146.1, 90.8)
- added SW1: SW_PUSH, footprint:switch, F.Cu at (127.6, 90.8)
- added SW1: SW_PUSH, footprint:switch, F.Cu at (109.2, 90.8)
- added SW1: SW_PUSH, footprint:switch, F.Cu at (90.8, 90.8)
- added SW1: SW_PUSH, footprint:switch, F.Cu at (146.1, 72.4)
- added SW1: SW_PUSH, footprint:switch, F.Cu at (127.6, 72.4)
- added SW1: SW_PUSH, footprint:switch, F.Cu at (109.2, 72.4)
- added SW1: SW_PUSH, footprint:switch, F.Cu at (90.8, 72.4)
- added SW1: SW_PUSH, footprint:switch, F.Cu at (146.1, 54.0)
- added SW1: SW_PUSH, footprint:switch, F.Cu at (164.5, 127.6)
- added SW1: SW_PUSH, footprint:switch, F.Cu at (127.6, 54.0)
- added SW1: SW_PUSH, footprint:switch, F.Cu at (109.2, 54.0)
- added SW1: SW_PUSH, footprint:switch, F.Cu at (146.1, 127.6)
- added SW1: SW_PUSH, footprint:switch, F.Cu at (127.6, 127.6)
- added SW1: SW_PUSH, footprint:switch, F.Cu at (109.2, 127.6)
- added SW1: SW_PUSH, footprint:switch, F.Cu at (90.8, 127.6)
- added SW1: SW_PUSH, footprint:switch, F.Cu at (146.1, 109.2)
- added SW1: SW_PUSH, footprint:switch, F.Cu at (127.6, 109.2)
- added SW1: SW_PUSH, footprint:switch, F.Cu at (109.2, 109.2)
- added U1: SK6812mini, sk6812:SK6812MINI_rev, F.Cu at (164.6, 113.7)
- added U1: SK6812mini, sk6812:SK6812MINI_rev, F.Cu at (90.9, 113.7)
- added U1: SK6812mini, sk6812:SK6812MINI_rev, F.Cu at (146.2, 95.3)
- added U1: SK6812mini, sk6812:SK6812MINI_rev, F.Cu at (127.8, 95.3)
- added U1: SK6812mini, sk6812:SK6812MINI_rev, F.Cu at (109.4, 95.3)
- added U1: SK6812mini, sk6812:SK6812MINI_rev, F.Cu at (90.9, 95.3)
- added U1: SK6812mini, sk6812:SK6812MINI_rev, F.Cu at (146.2, 76.9)
- added U1: SK6812mini, sk6812:SK6812MINI_rev, F.Cu at (127.8, 76.9)
- added U1: SK6812mini, sk6812:SK6812MINI_rev, F.Cu at (109.4, 76.9)
- added U1: SK6812mini, sk6812:SK6812MINI_rev, F.Cu at (90.9, 76.9)
- added U1: SK6812mini, sk6812:SK6812MINI_rev, F.Cu at (146.2, 58.5)
- added U1: SK6812mini, sk6812:SK6812MINI_rev, F.Cu at (164.6, 132.2)
- added U1: SK6812mini, sk6812:SK6812MINI_rev, F.Cu at (127.8, 58.5)
- added U1: SK6812mini, sk6812:SK6812MINI_rev, F.Cu at (109.4, 58.5)
- added U1: SK6812mini, sk6812:SK6812MINI_rev, F.Cu at (90.9, 58.5)
- added U1: SK6812mini, sk6812:SK6812MINI_rev, F.Cu at (146.2, 132.2)
- added U1: SK6812mini, sk6812:SK6812MINI_rev, F.Cu at (127.8, 132.2)
- added U1: SK6812mini, sk6812:SK6812MINI_rev, F.Cu at (109.4, 132.2)
- added U1: SK6812mini, sk6812:SK6812MINI_rev, F.Cu at (90.9, 132.2)
- added U1: SK6812mini, sk6812:SK6812MINI_rev, F.Cu at (146.2, 113.7)
- added U1: SK6812mini, sk6812:SK6812MINI_rev, F.Cu at (127.8, 113.7)
- added U1: SK6812mini, sk6812:SK6812MINI_rev, F.Cu at (109.4, 113.7)
- added U2: ProMicro, MYLIB:ProMicro_rev, B.Cu at (165.7, 62.9)
- moved P23 64.6 mm to (83.2, 46.4)
- moved P11 60.3 mm to (88.3, 46.4)
- moved P24 60.0 mm to (83.2, 56.5)
- moved D1 59.7 mm to (91.4, 46.4)
- moved SW1 59.7 mm to (90.8, 54.0)
- moved P21 59.4 mm to (98.4, 56.5)
- moved P22 59.4 mm to (98.4, 51.4)
- moved P14 59.4 mm to (83.2, 61.6)
- moved P13 59.1 mm to (88.3, 61.6)
- moved P16 59.1 mm to (93.3, 61.6)
- moved P15 58.9 mm to (98.4, 61.6)
- moved P12 55.9 mm to (83.2, 51.4)
Connections:
- P12 pad 1: /1 -> Net-(U1-Pad3)
- P14 pad 1: /1 -> Net-(U1-Pad2)
- P15 pad 1: /1 -> Net-(U1-Pad4)
- P16 pad 1: /1 -> Net-(U1-Pad2)
- P21 pad 1: /2 -> Net-(U1-Pad3)
- P24 pad 1: /2 -> Net-(U1-Pad1)
Routing:
- net Net-(U1-Pad2): track 0.00 -> 619.1 mm
- net Net-(U1-Pad3): track 0.00 -> 504.4 mm
- net /1: track 15.0 -> 478.1 mm
- net /2: track 21.2 -> 417.1 mm
- net Net-(U1-Pad4): track 0.00 -> 132.0 mm
- net Net-(U1-Pad1): track 0.00 -> 128.0 mm
- net Net-(D1-Pad2): track 5.87 -> 129.1 mm
- net GND: track 0.00 -> 85.2 mm
- net VCC: track 0.00 -> 81.4 mm
- net DATA: track 0.00 -> 71.9 mm
- net (no net): track 0.00 -> 47.9 mm
- net RESET: track 0.00 -> 41.7 mm
- net SCL: track 0.00 -> 30.8 mm
- net SDA: track 0.00 -> 29.5 mm
- net Net-(PM21-Pad1): track 0.00 -> 5.72 mm
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- added copper zone on F.Cu, net /1
- added copper zone on B.Cu, net /2
- added copper zone on F.Cu, net DATA
- added copper zone on B.Cu, net GND
- added copper zone on F.Cu, net Net-(D1-Pad2)
- added copper zone on B.Cu, net Net-(U1-Pad1)
- added copper zone on B.Cu, net Net-(U1-Pad2)
- added copper zone on F.Cu, net Net-(U1-Pad2)
- added copper zone on B.Cu, net Net-(U1-Pad3)
- added copper zone on B.Cu, net Net-(U1-Pad4)
- added copper zone on F.Cu, net SCL
- added copper zone on F.Cu, net SDA
- added copper zone on B.Cu, net VCC
Other:
- board size 17.8 x 17.8 mm -> 94 x 91.4 mm
- board text added: "+"
- board text added: "-"
- board text added: "10"
- board text added: "14"
- board text added: "15"
- board text added: "16"
- board text added: "4"
- board text added: "5"
- board text added: "6"
- board text added: "7"
- board text added: "8"
- board text added: "9"
- board text added: "A0"
- board text added: "A1"
- board text added: "A2"
- board text added: "A3"
- board text added: "C"
- board text added: "DI"
- board text added: "DO"
- board text added: "DT"
- board text added: "LED"
- board text added: "R"
- board text added: "RST"
- board text added: "SCL"
- board text added: "SDA"
- board text added: "SHIROTRON"
- board text added: "SwanMatch"
- board text removed: "1"
- board text removed: "2"
