File: Cherry Mx Bitboard.sch (KiCad schematic (older format))
At the start: 12 parts, among them P11 CONN_01X01, P12 CONN_01X01, P13 CONN_01X01, P14 CONN_01X01, P15 CONN_01X01, P16 CONN_01X01, P21 CONN_01X01, P22 CONN_01X01, P23 CONN_01X01, P24 CONN_01X01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

Commit message: first orderd
Parts:
- added J1: MJ-4PP-9, helix:MJ-4PP-9_rev2, symbol MJ-4PP-9
- added P1: OLED, helix:MY_SIL-4, symbol CONN_01X04
- added PLED1, PM10, PM14, PM15, PM16, PM18, PM19, PM20, PM21, PM4, PM5, PM6, PM7, PM8, PM9: CONN_01X01, footprint:wirepad, symbol Conn_01x01
- added RESET1: SW_PUSH, helix:SW_3.5x6.0_TH, symbol SW_PUSH
- added U1: SK6812mini, sk6812:SK6812MINI_rev, symbol SK6812mini
- added U2: ProMicro, promicro:ProMicro_rev, symbol ProMicro
- P11, P12, P13, P14, P15, P16, P21, P22, P23, P24: symbol CONN_01X01 -> Conn_01x01
Connections:
- net labels added: DATA, DI, DO, GND, RESET, SCL, SDA, VCC, VDD
- wire segments 13 -> 40
- no-connect marks 0 -> 1
Other:
- moved on the sheet: D1, SW1
