File: MxLEDBitPCB-promicro/MxLEDBit.kicad_pcb (KiCad board)
At the start: 2 copper layers, 85.1 x 54 mm, 276 parts, among them P2 CONN_01X01, U2 ProMicro

Commit message: git is difficult for me...
Parts:
- removed the JACK at (111.1, 91.9)
- removed the JACK at (132.7, 91.9)
- removed the JACK at (154.3, 91.9)
- removed the JACK at (175.8, 91.9)
- added JACK: MJ-4PP-9, helix:MJ-4PP-9_rev2, F.Cu at (175.9, 91.9)
- added JACK: MJ-4PP-9, helix:MJ-4PP-9_rev2, F.Cu at (154.3, 91.9)
- added JACK: MJ-4PP-9, helix:MJ-4PP-9_rev2, F.Cu at (132.7, 91.9)
- added JACK: MJ-4PP-9, helix:MJ-4PP-9_rev2, F.Cu at (111.1, 91.9)
Routing:
- net SDA: track 161.5 -> 118.7 mm
- net DATA: track 338.4 -> 302.8 mm
- net SCL: track 137.9 -> 104.3 mm
- net GND: track 348.6 -> 341.0 mm
- removed copper zone on F.Cu, net DATA
Other:
- net class VCC added: clearance 0.254, trace_width 1, via_dia 0.8, via_drill 0.4
