File: MxLEDBitPCB-promicro/promicro-home.kicad_pcb (KiCad board)
At the start: 2 copper layers, 85.1 x 54 mm, 276 parts, among them P2 CONN_01X01, U2 ProMicro

Commit message: ouchi_v2
Connections:
- HOLE_M2 pad : (no net) -> GND (x16)
Routing:
- net GND: vias 0 -> 4
- removed copper zone on B.Cu, net VCC
Other:
- board text added: "EndGame?"
- board text added: "Hack Kbd!!"
- board text removed: "SwanMatch"
