File: choc/choc.kicad_pcb (KiCad board)
At the start: 2 copper layers, 88.5 x 84 mm, 375 parts, among them SW1 SW_PUSH

Commit message: fix silk
Parts:
- L1: footprint keyboard:YS-SK6812MINI-E -> Keyboard:YS-SK6812MINI-E
Changed lines of the file:
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@@
-(kicad_pcb (version 20171130) (host pcbnew 5.0.2-bee76a0~70~ubuntu18.04.1)
+(kicad_pcb (version 20171130) (host pcbnew 5.1.5+dfsg1-2build2)
   (general
     (thickness 1.6)
@@
     (zone_45_only no)
     (trace_min 0.2)
-    (segment_width 0.2)
-    (edge_width 0.1)
     (via_size 0.6)
     (via_drill 0.4)
@@
     (uvia_min_size 0.2)
     (uvia_min_drill 0.1)
+    (edge_width 0.1)
+    (segment_width 0.2)
     (pcb_text_width 0.3)
     (pcb_text_size 1.5 1.5)
@@
     (add_net VCC)
   )
+  (module Keyboard:YS-SK6812MINI-E (layer B.Cu)
+    (at 74.422 31.002 180)
+    (fp_text reference L1 (at 0 -4.05 180) (layer B.SilkS)
+      (effects (font (size 1 1) (thickness 0.15)) (justify mirror))
+    )
+    (fp_text value SK6812MINI (at 0 -4.2 180) (layer B.Fab)
+      (effects (font (size 1 1) (thickness 0.15)) (justify mirror))
+    )
+    (fp_poly (pts (xy -3.81 -1.016) (xy -2.794 -2.032) (xy -3.81 -2.032)) (layer B.SilkS) (width 0.15))
+    (fp_line (start -1.7 1.5) (end -1.7 -1.5) (layer Edge.Cuts) (width 0.12))
+    (fp_line (start -1.7 -1.5) (end 1.7 -1.5) (layer Edge.Cuts) (width 0.12))
+    (fp_line (start 1.7 -1.5) (end 1.7 1.5) (layer Edge.Cuts) (width 0.12))
+    (fp_line (start 1.7 1.5) (end -1.7 1.5) (layer Edge.Cuts) (width 0.12))
+    (fp_text user V (at 4 0.75 180) (layer Dwgs.User)
+      (effects (font (size 1 1) (thickness 0.15)))
+    )
+    (fp_text user O (at 4 -0.75 180) (layer Dwgs.User)
+      (effects (font (size 1 1) (thickness 0.15)))
+    )
+    (fp_text user I (at -4 0.75 180) (layer Dwgs.User)
+      (effects (font (size 1 1) (thickness 0.15)))
+    )
+    (fp_text user G (at -4 -0.75 180) (layer Dwgs.User)
+      (effects (font (size 1 1) (thickness 0.15)))
+    )
+    (fp_line (start -3.5 1.5) (end -3.5 -1.5) (layer B.CrtYd) (width 0.12))
+    (fp_line (start -3.5 -1.5) (end 3.5 -1.5) (layer B.CrtYd) (width 0.12))
+    (fp_line (start 3.5 -1.5) (end 3.5 1.5) (layer B.CrtYd) (width 0.12))
+    (fp_line (start 3.5 1.5) (end -3.5 1.5) (layer B.CrtYd) (width 0.12))
+    (pad 4 smd rect (at -2.5 0.75 180) (size 1.8 0.82) (layers B.Cu B.Paste B.Mask)
+      (net 3 "Net-(L1-Pad3)"))
+    (pad 3 smd rect (at -2.5 -0.75 180) (size 1.8 0.82) (layers B.Cu B.Paste B.Mask)
+      (net 5 GND))
+    (pad 2 smd rect (at 2.5 -0.75 180) (size 1.8 0.82) (layers B.Cu B.Paste B.Mask)
+      (net 4 "Net-(L1-Pad1)"))
+    (pad 1 smd rect (at 2.5 0.75 180) (size 1.8 0.82) (layers B.Cu B.Paste B.Mask)
+      (net 7 VCC))
+  )
   (module keyboard:YS-SK6812MINI-E (layer B.Cu)
     (at 110.422 31.002 180)
@@
     (fp_text reference L1 (at 0 -4.05 180) (layer B.SilkS)
       (effects (font (size 1 1) (thickness 0.15)) (justify mirror))
-    )
-    (fp_text value SK6812MINI (at 0 -4.2 180) (layer B.Fab)
-      (effects (font (size 1 1) (thickness 0.15)) (justify mirror))
-    )
-    (fp_poly (pts (xy -3.683 -1.016) (xy -3.175 -1.524) (xy -3.683 -1.524)) (layer B.SilkS) (width 0.15))
-    (fp_line (start -1.7 1.5) (end -1.7 -1.5) (layer Edge.Cuts) (width 0.12))
-    (fp_line (start -1.7 -1.5) (end 1.7 -1.5) (layer Edge.Cuts) (width 0.12))
-    (fp_line (start 1.7 -1.5) (end 1.7 1.5) (layer Edge.Cuts) (width 0.12))
-    (fp_line (start 1.7 1.5) (end -1.7 1.5) (layer Edge.Cuts) (width 0.12))
-    (fp_text user V (at 4 0.75 180) (layer Dwgs.User)
-      (effects (font (size 1 1) (thickness 0.15)))
-    )
-    (fp_text user O (at 4 -0.75 180) (layer Dwgs.User)
-      (effects (font (size 1 1) (thickness 0.15)))
-    )
-    (fp_text user I (at -4 0.75 180) (layer Dwgs.User)
-      (effects (font (size 1 1) (thickness 0.15)))
-    )
-    (fp_text user G (at -4 -0.75 180) (layer Dwgs.User)
-      (effects (font (size 1 1) (thickness 0.15)))
-    )
-    (fp_line (start -3.5 1.5) (end -3.5 -1.5) (layer B.CrtYd) (width 0.12))
-    (fp_line (start -3.5 -1.5) (end 3.5 -1.5) (layer B.CrtYd) (width 0.12))
-    (fp_line (start 3.5 -1.5) (end 3.5 1.5) (layer B.CrtYd) (width 0.12))
-    (fp_line (start 3.5 1.5) (end -3.5 1.5) (layer B.CrtYd) (width 0.12))
-    (pad 4 smd rect (at -2.5 0.75 180) (size 1.8 0.82) (layers B.Cu B.Paste B.Mask)
-      (net 3 "Net-(L1-Pad3)"))
-    (pad 3 smd rect (at -2.5 -0.75 180) (size 1.8 0.82) (layers B.Cu B.Paste B.Mask)
-      (net 5 GND))
-    (pad 2 smd rect (at 2.5 -0.75 180) (size 1.8 0.82) (layers B.Cu B.Paste B.Mask)
-      (net 4 "Net-(L1-Pad1)"))
-    (pad 1 smd rect (at 2.5 0.75 180) (size 1.8 0.82) (layers B.Cu B.Paste B.Mask)
-      (net 7 VCC))
-  )
-  (module keyboard:YS-SK6812MINI-E (layer B.Cu)
-    (at 74.422 31.002 180)
-    (fp_text reference L1 (at 0 -4.05 180) (layer B.SilkS)
-      (effects (font (size 1 1) (thickness 0.15)) (justify mirror))
