File: suxen/suxen.kicad_pcb (KiCad board)
At the start: 2 copper layers, 94 x 94 mm, 375 parts, among them SW1 SW_PUSH, SW10 SW_PUSH, SW11 SW_PUSH, SW12 SW_PUSH, SW13 SW_PUSH, SW14 SW_PUSH, SW15 SW_PUSH, SW16 SW_PUSH, SW17 SW_PUSH, SW18 SW_PUSH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

Commit message: fix silk
Parts:
- L1 (x25): footprint keyboard:YS-SK6812MINI-E -> Keyboard:YS-SK6812MINI-E
