File: altana/altana.kicad_pcb (KiCad board)
At the start: 2 copper layers, 94 x 94 mm, 375 parts, among them SW1 SW_PUSH, SW10 SW_PUSH, SW11 SW_PUSH, SW12 SW_PUSH, SW13 SW_PUSH, SW14 SW_PUSH, SW15 SW_PUSH, SW16 SW_PUSH, SW17 SW_PUSH, SW18 SW_PUSH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

Commit message: nexus and altana
Routing:
- net /ROW0: track 207.2 -> 201.7 mm, vias 11 -> 10
- net /COL4: track 112.3 -> 117.0 mm
- net GND: vias 0 -> 175
- net VCC: vias 25 -> 75
- removed copper zone on B.Cu, net (none)
- removed copper zone on F.Cu, net (none)

Commit message: Enlarge the connection bits to at least 4mm
Other:
- outline, holes or cut-outs redrawn
